File: hardware/MaoRad.kicad_sch (KiCad schematic)
At the start: 24 parts, among them J1 Conn, Q1 MMBT3904, U1 LMC6062, U2 LM1117-5.0

Commit message: fix: lmc662
Parts:
- U1: value LMC6062 -> LMC662; footprint (none) -> Package_SO:SOIC-8_3.9x4.9mm_P1.27mm
- U1: value LMC6062 -> LMC662
Changed lines of the file:
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@@
     (in_bom yes) (on_board yes)
     (property "Reference" "U1" (id 0) (at 146.05 111.76 0))
-    (property "Value" "LMC6062" (id 1) (at 146.05 114.3 0))
-    (property "Footprint" "" (id 2) (at 142.24 119.38 0)
+    (property "Value" "LMC662" (id 1) (at 146.05 114.3 0))
+    (property "Footprint" "Package_SO:SOIC-8_3.9x4.9mm_P1.27mm" (id 2) (at 142.24 119.38 0)
       (effects (font (size 1.27 1.27)) hide)
     )
@@
       (effects (font (size 1.27 1.27)) (justify left) hide)
     )
-    (property "Value" "LMC6062" (id 1) (at 140.97 120.6499 0)
+    (property "Value" "LMC662" (id 1) (at 140.97 120.6499 0)
       (effects (font (size 1.27 1.27)) (justify left) hide)
     )
@@
     (in_bom yes) (on_board yes) (fields_autoplaced)
     (property "Reference" "U1" (id 0) (at 185.42 111.76 0))
-    (property "Value" "LMC6062" (id 1) (at 185.42 114.3 0))
+    (property "Value" "LMC662" (id 1) (at 185.42 114.3 0))
     (property "Footprint" "Package_SO:SOIC-8_3.9x4.9mm_P1.27mm" (id 2) (at 185.42 121.92 0)
       (effects (font (size 1.27 1.27)) hide)
@@
     )
     (path "/10e17507-bb2c-4af8-8356-394af0f548c7"
-      (reference "U1") (unit 1) (value "LMC6062") (footprint "Package_SO:SOIC-8_3.9x4.9mm_P1.27mm")
+      (reference "U1") (unit 1) (value "LMC662") (footprint "Package_SO:SOIC-8_3.9x4.9mm_P1.27mm")
     )
     (path "/1b3735e4-6f49-4924-90f5-9f892e631ceb"
-      (reference "U1") (unit 2) (value "LMC6062") (footprint "Package_SO:SOIC-8_3.9x4.9mm_P1.27mm")
+      (reference "U1") (unit 2) (value "LMC662") (footprint "Package_SO:SOIC-8_3.9x4.9mm_P1.27mm")
     )
     (path "/182ab6bc-e765-40b2-b4fa-9edeb4467222"
-      (reference "U1") (unit 3) (value "LMC6062") (footprint "Package_SO:SOIC-8_3.9x4.9mm_P1.27mm")
+      (reference "U1") (unit 3) (value "LMC662") (footprint "Package_SO:SOIC-8_3.9x4.9mm_P1.27mm")
     )
     (path "/9dd6d4cf-af95-450a-8849-bd2f685f898c"
